File: hardware/pcb/hub_v1.5/kicad/blackout_sensor_hub.kicad_pcb (KiCad board)
At the start: 2 copper layers, 101.6 x 53.3 mm, 63 parts, among them J1 GIGA_POWER, J10 ARM_PCA9685, J11 LCD_ILI9488_SPI, J12 BME280, J13 Qwiic_I2C1, J14 Qwiic_I2C1, J15 GY-302_BH1750, J16 Qwiic_I2C2, J17 Qwiic_I2C2, J18 RCWL-1601, J19 DHT11, J2 GIGA_D8-D13_I2C1, J20 BUZZER, J21 RELAYS, J22 L298N, J23 LIDAR_UART3, J24 LIDAR_PWM, J25 IMU_UART4, J27 Qwiic_I2C2, J28 AUX_3P, J29 AUX_4P, J3 GIGA_A0-A7, J30 GPIO_BREAKOUT, J31 3V3_GND_RAIL, J32 GYRO_I2C1, J33 MQ135, J4 GIGA_D0-D7, J5 GIGA_A8-A11_DAC_CAN, J6 GIGA_D14-D21, J7 GIGA_D22-D53

Commit message: feat(pcb): hub v1.6 — NEO-7M GPS on J28 (UART2 D19/D18), drop A0
Parts:
- added R14: 1k, Resistor_SMD:R_0805_2012Metric_Pad1.20x1.40mm_HandSolder, F.Cu at (168.5, 76.0)
- J28: value AUX_3P -> GPS_NEO-7M; footprint Connector_JST:JST_PH_B3B-PH-SM4-TB_1x03-1MP_P2.00mm_Vertical -> Connector_JST:JST_PH_B4B-PH-SM4-TB_1x04-1MP_P2.00mm_Vertical
- moved J28 1.92 mm to (162.6, 81.0), turned to -90 degrees
Connections:
- J28 pad 2: GPIO_A0 -> GND
- J28 pad 3: GND -> GPS_TXO
- J3 pad 1: GPIO_A0 -> unconnected-(J3-Pin_1-Pad1)
Routing:
- net UART2_RX: track 69.5 -> 118.7 mm, vias 0 -> 1
- net UART2_TX: track 74.3 -> 113.9 mm, vias 1 -> 3
- net GPIO_A0: track 36.3 -> 0.00 mm, vias 2 -> 0
- net BUZZ_D34: track 57.8 -> 76.9 mm, vias 0 -> 4
- net SONAR_ECHO: track 89.6 -> 101.4 mm, vias 2 -> 3
- net +3V3: track 369.9 -> 360.3 mm
- net GPS_TXO: track 0.00 -> 8.60 mm
- net GND: track 537.9 -> 539.3 mm, vias 248 -> 233
Other:
- board text added: "GPS UART2 D18/D19 AUX D44/46 MQ135 A1 GYRO W1"
- board text added: "GPS UART2 D19"
- board text removed: "AUX A0"
- board text removed: "AUX A0, D44/46 MQ135 A1 GYRO ON W1"
