File: hardware/pcb/hub_v1.5/kicad/blackout_sensor_hub.kicad_sch (KiCad schematic)
At the start: 63 parts, among them J1 GIGA_POWER, J10 ARM_PCA9685, J11 LCD_ILI9488_SPI, J12 BME280, J13 Qwiic_I2C1, J14 Qwiic_I2C1, J15 GY-302_BH1750, J16 Qwiic_I2C2, J17 Qwiic_I2C2, J18 RCWL-1601, J19 DHT11, J2 GIGA_D8-D13_I2C1, J20 BUZZER, J21 RELAYS, J22 L298N, J23 LIDAR_UART3, J24 LIDAR_PWM, J25 IMU_UART4, J27 Qwiic_I2C2, J28 AUX_3P, J29 AUX_4P, J3 GIGA_A0-A7, J30 GPIO_BREAKOUT, J31 3V3_GND_RAIL, J32 GYRO_I2C1, J33 MQ135, J4 GIGA_D0-D7, J5 GIGA_A8-A11_DAC_CAN, J6 GIGA_D14-D21, J7 GIGA_D22-D53

Commit message: feat(pcb): hub v1.6 — NEO-7M GPS on J28 (UART2 D19/D18), drop A0
Parts:
- added R14: 1k, Resistor_SMD:R_0805_2012Metric_Pad1.20x1.40mm_HandSolder, symbol Device:R
- J28: value AUX_3P -> GPS_NEO-7M; footprint Connector_JST:JST_PH_B3B-PH-SM4-TB_1x03-1MP_P2.00mm_Vertical -> Connector_JST:JST_PH_B4B-PH-SM4-TB_1x04-1MP_P2.00mm_Vertical; symbol Connector_Generic_MountingPin:Conn_01x03_MountingPin -> Connector_Generic_MountingPin:Conn_01x04_MountingPin; LCSC C160353 -> C160354; MPN JST B3B-PH-SM4-TB(LF)(SN) -> JST B4B-PH-SM4-TB(LF)(SN)
Connections:
- net GND: now also J28.2 (Pin_2); no longer J28.3 (Pin_3)
- net UART2_RX: now also R14.2
- net UART2_TX: now also J28.4 (Pin_4)
- net GPIO_A0: no longer names the net of J3.1 (Pin_1)
- net GPIO_A0: no longer J28.2 (Pin_2)
- new net GPS_TXO: J28.3 (Pin_3), R14.1
- no-connect marks 40 -> 41
Other:
- moved on the sheet: H1, H2, H3, H4, H5, H6, J29, J32, J33, R12, R13
